Commit message: adding simulated world and open rviz and gazebo in same time

File: diff_bot/urdf/lidar.xacro (robot description, xacro)
@@ -12,5 +12,5 @@
   <!-- Fixed Joint to Mount LiDAR -->
   <joint name="laser_joint" type="fixed">
-    <origin xyz="0 0 0.15" rpy="0 0 0"/>
+    <origin xyz="0 0 0.08" rpy="0 0 0"/>
     <parent link="chassis_link"/> <!-- Make sure chassis_link is defined elsewhere -->
     <child link="laser_frame"/>
@@ -21,5 +21,5 @@
     <sensor name="laser" type="ray">
       <pose>0 0 0.1 0 0 0</pose>
-      <visualize>true</visualize>
+      <visualize>false</visualize>
       <update_rate>30.0</update_rate>
       <ray>
