Commit message: navigation_problems still not done

File: diff_bot/urdf/caster_wheel.xacro (robot description, xacro)
@@ -50,6 +50,6 @@
       </joint>
       <gazebo reference="caster_wheel_link">
-        <mu1>0.001</mu1>
-        <mu2>0.002</mu2>
+        <mu1 value="0.001"/>
+        <mu2 value="0.002"/>
       </gazebo>
 </robot>

File: diff_bot/urdf/chassis.xacro (robot description, xacro)
@@ -11,16 +11,16 @@
         <visual>
             <geometry>
-                <box size="0.4 0.3 0.1"/>
-                <origin xyz="0.2 0.0 0.05" rpy="0.0 0.0 0.0"/>
+                <box size="${chassis_length} ${chassis_width} ${chassis_height}"/>
+                <origin xyz="${chassis_length/2} 0.0 ${chassis_height/2}" rpy="0.0 0.0 0.0"/>
             </geometry>
         </visual>
         <collision>
             <geometry>
-                <box size="0.4 0.3 0.1"/>
-                <origin xyz="0.2 0.0 0.05" rpy="0.0 0.0 0.0"/>
+                <box size="${chassis_length} ${chassis_width} ${chassis_height}"/>
+                <origin xyz="${chassis_length/2} 0.0 ${chassis_height/2}" rpy="0.0 0.0 0.0"/>
             </geometry>
         </collision>
         <xacro:inertial_box mass="2" x="0.4" y="0.3" z="0.11"/>
-        <origin xyz="0.2 0.0 0.05" rpy="0.0 0.0 0.0"/>
+        <origin xyz="${chassis_length/2} 0.0 ${chassis_height/2}" rpy="0.0 0.0 0.0"/>
     </link>
     <joint name="chassis_joint" type="fixed">

File: diff_bot/urdf/control.xacro (robot description, xacro)
@@ -1,2 +1,3 @@
+<?xml version="1.0"?>
 <robot xmlns:xacro="http://www.ros.org/wiki/xacro">
   <ros2_control name="DiffBot" type="system">
@@ -9,20 +10,23 @@
       <param name="timeout">0.5</param>
       <param name="baud_rate">57600</param>
-      <param name="encoder_resolution">500</param>
-      <param name="ticks_per_rev">1500</param>
+      <!-- <param name="encoder_resolution">500</param> -->
+      <!-- <param name="ticks_per_rev">1500</param> -->
+       <param name="enc_counts_per_rev">1500</param>
     </hardware>
     <joint name="left_wheel_joint">
-      <command_interface name="velocity"/>
+      <command_interface name="velocity">
+        <param name="min">-10</param>
+        <param name="max">10</param>
+      </command_interface>
       <state_interface name="position"/>
       <state_interface name="velocity"/>
-      <param name="min">-10</param>
-      <param name="max">10</param>
     </joint>
     <joint name="right_wheel_joint">
-      <command_interface name="velocity"/>
+      <command_interface name="velocity">
+        <param name="min">-10</param>
+        <param name="max">10</param>
+      </command_interface>
       <state_interface name="position"/>
       <state_interface name="velocity"/>
-      <param name="min">-10</param>
-      <param name="max">10</param>
     </joint>
   </ros2_control>

File: diff_bot/urdf/lidar.xacro (robot description, xacro)
@@ -12,5 +12,5 @@
   <!-- Fixed Joint to Mount LiDAR -->
   <joint name="laser_joint" type="fixed">
-    <origin xyz="0 0 0.08" rpy="0 0 0"/>
+    <origin xyz="0.0 0 0.08" rpy="0 0 0"/>
     <parent link="chassis_link"/> <!-- Make sure chassis_link is defined elsewhere -->
     <child link="laser_frame"/>
@@ -22,5 +22,5 @@
       <pose>0 0 0.1 0 0 0</pose>
       <visualize>false</visualize>
-      <update_rate>30.0</update_rate>
+      <update_rate>100.0</update_rate>
       <ray>
         <scan>

File: diff_bot/urdf/properties.xacro (robot description, xacro)
@@ -3,5 +3,5 @@
     <!-- Chassis -->
     <xacro:property name="chassis_length" value="0.4"/>
-    <xacro:property name="chassis_width" value="0.3"/>
+    <xacro:property name="chassis_width" value="0.4"/>
     <xacro:property name="chassis_height" value="0.11"/>
     <xacro:property name="chassis_mass" value="2.0"/>
