Commit message: BASH FILES WORKING

File: diff_bot/urdf/chassis.xacro (robot description, xacro)
@@ -12,5 +12,5 @@
             <geometry>
                 <box size="${chassis_length} ${chassis_width} ${chassis_height}"/>
-                <origin xyz="${chassis_length/2} 0.0 ${chassis_height/2}" rpy="0.0 0.0 0.0"/>
+                <origin xyz="${chassis_length/2} 0.0 ${chassis_height}" rpy="0.0 0.0 0.0"/>
             </geometry>
         </visual>
@@ -18,9 +18,9 @@
             <geometry>
                 <box size="${chassis_length} ${chassis_width} ${chassis_height}"/>
-                <origin xyz="${chassis_length/2} 0.0 ${chassis_height/2}" rpy="0.0 0.0 0.0"/>
+                <origin xyz="${chassis_length/2} 0.0 ${chassis_height}" rpy="0.0 0.0 0.0"/>
             </geometry>
         </collision>
         <xacro:inertial_box mass="2" x="0.4" y="0.3" z="0.11"/>
-        <origin xyz="${chassis_length/2} 0.0 ${chassis_height/2}" rpy="0.0 0.0 0.0"/>
+        <origin xyz="${chassis_length/2} 0.0 ${chassis_height}" rpy="0.0 0.0 0.0"/>
     </link>
     <joint name="chassis_joint" type="fixed">

File: diff_bot/urdf/properties.xacro (robot description, xacro)
@@ -3,6 +3,6 @@
     <!-- Chassis -->
     <xacro:property name="chassis_length" value="0.4"/>
-    <xacro:property name="chassis_width" value="0.4"/>
-    <xacro:property name="chassis_height" value="0.11"/>
+    <xacro:property name="chassis_width" value="0.3"/>
+    <xacro:property name="chassis_height" value="0.05"/>
     <xacro:property name="chassis_mass" value="2.0"/>
     <!-- Wheels -->
